File: PCB_Design/batteryCharge.sch (KiCad schematic (older format))
At the start: 11 parts, among them J1 TP4056, J2 USB_B_Micro

Commit message: PCB terminada
Parts:
- R_PROG1: value R -> 4.7k
Changed lines of the file:
@@
 P 3210 3175
 F 0 "R_PROG1" V 3125 3015 50  0000 L CNN
-F 1 "R" V 3215 3145 50  0000 L CNN
+F 1 "4.7k" V 3210 3090 50  0000 L CNN
 F 2 "Resistor_SMD:R_0805_2012Metric_Pad1.20x1.40mm_HandSolder" V 3140 3175 50  0001 C CNN
 F 3 "~" H 3210 3175 50  0001 C CNN
